Commit message: Update with usable gazebo

File: src/robot_description/urdf/materials.xacro (robot description, xacro)
@@ -1,4 +1,4 @@
 <?xml version="1.0" ?>
-<robot name="robot" xmlns:xacro="http://www.ros.org/wiki/xacro" >
+<robot xmlns:xacro="http://www.ros.org/wiki/xacro" >
 <material name="silver">
   <color rgba="0.700 0.700 0.700 1.000"/>

File: src/robot_description/urdf/robot.xacro (robot description, xacro)
@@ -3,5 +3,5 @@
 <xacro:include filename="$(find robot_description)/urdf/materials.xacro" />
 <xacro:include filename="$(find robot_description)/urdf/macros.xacro" />
-<xacro:include filename="$(find robot_description)/urdf/robot.trans" />
+<xacro:include filename="$(find robot_description)/urdf/robot.control" />
 <xacro:include filename="$(find robot_description)/urdf/robot.gazebo" />
 <!-- Properties -->
@@ -10,5 +10,5 @@
 <xacro:property name="chassis_height" value="0.135" />
 <xacro:property name="chassis_weight" value="2.45" />
-<xacro:property name="wheel_radius" value="0.0466" />
+<xacro:property name="wheel_radius" value="0.047" />
 <xacro:property name="wheel_thickness" value="0.042" />
 <xacro:property name="wheel_weight" value=".136" />
@@ -17,4 +17,10 @@
 <xacro:property name="joint_pos_z" value="0.121" />
 <!-- Links -->
+<link name="base_link"></link>
+<joint name="chassis_joint" type="fixed">
+  <parent link="base_link"/>
+  <child link="chassis"/>
+  <origin xyz="0 0 0"/>
+</joint>
 <link name="chassis">
   <xacro:inertial_box mass="${chassis_weight}" x="${chassis_length}" y="${chassis_width}" z="${chassis_height}">
