Commit message: Add isaac files

File: src/robot_description/urdf/mechanical/mecanum_with_rollers.urdf.xacro (robot description, xacro)
@@ -7,40 +7,7 @@
       </xacro:inertial_cylinder>
       <visual>
-        <origin xyz="0 0 0" rpy="0 ${(type - 1) * (pi/2)} 0"/>
-        <geometry>
-          <mesh filename="package://robot_description/meshes/mecanum_${type}.stl" scale="0.001 0.001 0.001"/>
-        </geometry>
-        <material name="silver"/>
-      </visual>
-    </link>
-    <joint name="${name}_mecanum_joint" type="continuous">
-      <origin xyz="${pos_x} ${pos_y} ${pos_z}" rpy="0 ${flip} 0"/>
-      <parent link="chassis_link"/>
-      <child link="${name}_mecanum_link"/>
-      <axis xyz="1.0 0.0 0.0"/>
-    </joint>
-    <xacro:roller name="${name}" number="0" center="-${width/2}"/>
-    <xacro:roller name="${name}" number="1" center="-${width/2}"/>
-    <xacro:roller name="${name}" number="2" center="-${width/2}"/>
-    <xacro:roller name="${name}" number="3" center="-${width/2}"/>
-    <xacro:roller name="${name}" number="4" center="-${width/2}"/>
-    <xacro:roller name="${name}" number="5" center="-${width/2}"/>
-    <xacro:roller name="${name}" number="6" center="-${width/2}"/>
-    <xacro:roller name="${name}" number="7" center="-${width/2}"/>
-    <xacro:roller name="${name}" number="8" center="-${width/2}"/>
-  </xacro:macro>
-  <xacro:macro name="roller" params="name number center">
-    <xacro:property name="diff" value="0.002" />
-    <xacro:property name="roller_radius" value="${radius - diff}" />
-    <xacro:property name="roller_total" value="9" />
-    <xacro:property name="roller_radians" value="${2 * pi / roller_total * number}" />
-    <xacro:property name="roller_y" value="${sin(roller_radians) * diff}" />
-    <xacro:property name="roller_z" value="${cos(roller_radians) * diff}" />
-    <xacro:property name="roller_axis" value="${((type - 1) * -1) + 0.5}" />
-    <link name="${name}_roller_${number}">
-      <visual>
         <origin xyz="0 0 0" rpy="0 0 0"/>
         <geometry>
-          <sphere radius="${roller_radius}"/>
+          <mesh filename="package://robot_description/meshes/mec_hub_${type}.stl" scale="0.001 0.001 0.001"/>
         </geometry>
         <material name="silver"/>
@@ -49,16 +16,83 @@
         <origin xyz="0 0 0" rpy="0 0 0"/>
         <geometry>
-          <sphere radius="${roller_radius}"/>
+          <cylinder radius="${radius}" length="${width}"/>
         </geometry>
       </collision>
-      <xacro:inertial_sphere mass="0.03" radius="${roller_radius}">
+    </link>
+    <joint name="${name}_mecanum_joint" type="continuous">
+      <origin xyz="${pos_x} ${pos_y} ${pos_z}" rpy="0 ${flip} 0"/>
+      <parent link="chassis_link"/>
+      <child link="${name}_mecanum_link"/>
+      <axis xyz="0.0 0.0 ${copysign(1, (flip * -1))}"/>
+    </joint>
+    <xacro:roller name="${name}" number="0" wheel_radius="${radius}"/>
+    <xacro:roller name="${name}" number="1" wheel_radius="${radius}"/>
+    <xacro:roller name="${name}" number="2" wheel_radius="${radius}"/>
+    <xacro:roller name="${name}" number="3" wheel_radius="${radius}"/>
+    <xacro:roller name="${name}" number="4" wheel_radius="${radius}"/>
+    <xacro:roller name="${name}" number="5" wheel_radius="${radius}"/>
+    <xacro:roller name="${name}" number="6" wheel_radius="${radius}"/>
+    <xacro:roller name="${name}" number="7" wheel_radius="${radius}"/>
+    <xacro:roller name="${name}" number="8" wheel_radius="${radius}"/>
+  </xacro:macro>
+  <xacro:property name="roller_middle_radius" value="${0.0194/2}" />
+  <xacro:property name="roller_second_radius" value="${0.01904/2}" />
+  <xacro:property name="roller_third_radius" value="${0.01797/2}" />
+  <xacro:property name="roller_cylinder_radius" value="0.0074" />
+  <xacro:property name="roller_length" value="0.0396" />
+  <xacro:macro name="roller" params="name number wheel_radius">
+    <!-- Type Negative: When 1 output 1. When 2 output -1 -->
+    <xacro:property name="type_negative" value="${(type * 2 - 3) * -1}" />
+    <xacro:property name="roller_total" value="9" />
+    <xacro:property name="roller_radians" value="${2 * pi / roller_total * number}" />
+    <xacro:property name="roller_x_pos" value="${sin(roller_radians) * wheel_radius}" />
+    <xacro:property name="roller_y_pos" value="${cos(roller_radians) * wheel_radius}" />
+    <xacro:property name="roller_x_rot" value="${sin(roller_radians) * (pi/4) * type_negative}" />
+    <xacro:property name="roller_y_rot" value="${cos(roller_radians) * (pi/4) * type_negative}" />
+    <xacro:property name="roller_z_rot" value="${tan(roller_radians) * (pi/4) * type_negative}" />
+    <link name="${name}_roller_${number}">
+      <visual>
         <origin xyz="0 0 0" rpy="0 0 0"/>
-      </xacro:inertial_sphere>
+        <geometry>
+          <mesh filename="package://robot_description/meshes/roller.stl" scale="0.001 0.001 0.001"/>
+        </geometry>
+        <material name="silver"/>
+      </visual>
+      <collision>
+        <origin xyz="0 0 0" rpy="0 0 0"/>
+        <geometry>
+          <sphere radius="${roller_middle_radius}"/>
+        </geometry>
+      </collision>
+      <collision>
+        <origin xyz="0 0 ${roller_length/5}" rpy="0 0 0"/>
+        <geometry>
+          <sphere radius="${roller_second_radius}"/>
+        </geometry>
+      </collision>
+      <collision>
+        <origin xyz="0 0 -${roller_length/5}" rpy="0 0 0"/>
+        <geometry>
+          <sphere radius="${roller_second_radius}"/>
+        </geometry>
+      </collision>
+      <collision>
+        <origin xyz="0 0 ${2 * roller_length/5}" rpy="0 0 0"/>
+        <geometry>
+          <sphere radius="${roller_third_radius}"/>
+        </geometry>
+      </collision>
+      <collision>
+        <origin xyz="0 0 -${2 * roller_length/5}" rpy="0 0 0"/>
+        <geometry>
+          <sphere radius="${roller_third_radius}"/>
+        </geometry>
+      </collision>
     </link>
     <joint name="${name}_roller_${number}_joint" type="continuous">
-      <origin xyz="${center} ${roller_y} ${roller_z}" rpy="0 ${roller_radians} 0"/>
+      <origin xyz="${roller_x_pos} ${roller_y_pos} 0" rpy="${roller_x_rot} ${roller_y_rot} 0"/>
       <parent link="${name}_mecanum_link"/>
       <child link="${name}_roller_${number}"/>
-      <axis xyz="0.5 ${roller_axis} 0.0"/>
+      <axis xyz="0.0 0.0 1.0"/>
     </joint>
   </xacro:macro>

File: src/robot_description/urdf/robots/examplo.urdf.xacro (robot description, xacro)
@@ -16,6 +16,6 @@
     radius="${wheel_radius}"
     width="${wheel_thickness}"
-    flip="${pi}"
-    pos_x="${wheel_joint_pos_x}"
+    flip="${pi/2}"
+    pos_x="${wheel_joint_pos_x + wheel_offset}"
     pos_y="${wheel_joint_pos_y}"
     pos_z="-${wheel_joint_pos_z}"
@@ -27,6 +27,6 @@
     radius="${wheel_radius}"
     width="${wheel_thickness}"
-    flip="0"
-    pos_x="-${wheel_joint_pos_x}"
+    flip="-${pi/2}"
+    pos_x="-${wheel_joint_pos_x + wheel_offset}"
     pos_y="-${wheel_joint_pos_y}"
     pos_z="-${wheel_joint_pos_z}"
@@ -38,6 +38,6 @@
     radius="${wheel_radius}"
     width="${wheel_thickness}"
-    flip="0"
-    pos_x="-${wheel_joint_pos_x}"
+    flip="${pi/2}"
+    pos_x="-${wheel_joint_pos_x + wheel_offset}"
     pos_y="${wheel_joint_pos_y}"
     pos_z="-${wheel_joint_pos_z}"
@@ -49,6 +49,6 @@
     radius="${wheel_radius}"
     width="${wheel_thickness}"
-    flip="${pi}"
-    pos_x="${wheel_joint_pos_x}"
+    flip="-${pi/2}"
+    pos_x="${wheel_joint_pos_x + wheel_offset}"
     pos_y="-${wheel_joint_pos_y}"
     pos_z="-${wheel_joint_pos_z}"

File: src/robot_description/urdf/robots/examplo_properties.urdf.xacro (robot description, xacro)
@@ -5,7 +5,8 @@
     <xacro:property name="chassis_height" value="0.135" />
     <xacro:property name="chassis_weight" value="2.45" />
-    <xacro:property name="wheel_radius" value="0.047" />
+    <xacro:property name="wheel_radius" value="${0.0194/2 + 0.0291}" />
     <xacro:property name="wheel_thickness" value="0.042" />
     <xacro:property name="wheel_weight" value="0.136" />
+    <xacro:property name="wheel_offset" value="${wheel_thickness/2 - 0.003}" />
     <xacro:property name="wheel_joint_pos_x" value="0.09" />
     <xacro:property name="wheel_joint_pos_y" value="0.145" />
