Commit message: Add robot hardware

File: src/robot_description/urdf/control/drive.xacro (robot description, xacro)
@@ -1,9 +1,11 @@
 <?xml version="1.0"?>
 <robot name="robot" xmlns:xacro="http://www.ros.org/wiki/xacro" >
-  <ros2_control name="robot" type="system">
+  <ros2_control name="examplo" type="system">
     <hardware>
-      <plugin>gazebo_ros2_control/GazeboSystem</plugin>
+      <plugin>robot_hardware/IsaacDriveHardware</plugin>
+      <param name="example_param_hw_start_duration_sec">3.0</param>
+      <param name="example_param_hw_stop_duration_sec">3.0</param>
     </hardware>
-    <joint name="wheel_FR_joint">
+    <joint name="front_right_mecanum_joint">
       <command_interface name="velocity">
         <param name="min">-1</param>
@@ -13,5 +15,5 @@
       <state_interface name="velocity"/>
     </joint>
-    <joint name="wheel_FL_joint">
+    <joint name="rear_left_mecanum_joint">
       <command_interface name="velocity">
         <param name="min">-1</param>
@@ -21,5 +23,5 @@
       <state_interface name="velocity"/>
     </joint>
-    <joint name="wheel_RR_joint">
+    <joint name="front_left_mecanum_joint">
       <command_interface name="velocity">
         <param name="min">-1</param>
@@ -29,5 +31,5 @@
       <state_interface name="velocity"/>
     </joint>
-    <joint name="wheel_RL_joint">
+    <joint name="rear_right_mecanum_joint">
       <command_interface name="velocity">
         <param name="min">-1</param>
@@ -38,8 +40,3 @@
     </joint>
   </ros2_control>
-  <gazebo>
-    <plugin filename="libgazebo_ros2_control.so" name="gazebo_ros2_control">
-      <parameters>$(find robot_description)/config/diff_drive_controller.yml</parameters>
-    </plugin>
-  </gazebo>
 </robot>

File: src/robot_description/urdf/parts/chassis.xacro (robot description, xacro)
@@ -12,5 +12,5 @@
           <mesh filename="package://robot_description/meshes/chassis.stl" scale="0.001 0.001 0.001"/>
         </geometry>
-        <material name="silver"/>
+        <material name="blue"/>
       </visual>
       <collision>

File: src/robot_description/urdf/robots/examplo.urdf.xacro (robot description, xacro)
@@ -1,8 +1,30 @@
 <?xml version="1.0" ?>
 <robot name="examplo" xmlns:xacro="http://www.ros.org/wiki/xacro">
-  <xacro:include filename="$(find robot_description)/urdf/macros.xacro" />
-  <xacro:include filename="$(find robot_description)/urdf/mechanical/chassis.urdf.xacro"/>
-  <xacro:include filename="$(find robot_description)/urdf/mechanical/mecanum_with_rollers.urdf.xacro"/>
-  <xacro:include filename="$(find robot_description)/urdf/robots/examplo_properties.urdf.xacro"/>
+  <!-- Include Files -->
+  <xacro:include filename="$(find robot_description)/urdf/util/macros.xacro" />
+  <xacro:include filename="$(find robot_description)/urdf/util/materials.xacro" />
+  <xacro:include filename="$(find robot_description)/urdf/parts/chassis.xacro"/>
+  <xacro:include filename="$(find robot_description)/urdf/parts/mecanum_wheel.xacro"/>
+  <xacro:include filename="$(find robot_description)/urdf/parts/mecanum_roller.xacro"/>
+  <xacro:include filename="$(find robot_description)/urdf/control/drive.xacro"/>
+  <!-- Properties -->
+  <xacro:property name="chassis_length" value="0.18" />
+  <xacro:property name="chassis_width" value="0.33" />
+  <xacro:property name="chassis_height" value="0.135" />
+  <xacro:property name="chassis_weight" value="2.45" />
+  <xacro:property name="wheel_radius" value="${0.0194/2 + 0.0291}" />
+  <xacro:property name="wheel_thickness" value="0.042" />
+  <xacro:property name="wheel_weight" value="0.136" />
+  <xacro:property name="wheel_offset" value="${wheel_thickness/2 - 0.003}" />
+  <xacro:property name="wheel_joint_pos_x" value="0.09" />
+  <xacro:property name="wheel_joint_pos_y" value="0.145" />
+  <xacro:property name="wheel_joint_pos_z" value="0.121" />
+  <xacro:property name="roller_total" value="9" />
+  <xacro:property name="roller_middle_radius" value="${0.0194/2}" />
+  <xacro:property name="roller_second_radius" value="${0.01904/2}" />
+  <xacro:property name="roller_third_radius" value="${0.01797/2}" />
+  <xacro:property name="roller_cylinder_radius" value="0.0074" />
+  <xacro:property name="roller_length" value="0.0396" />
+  <!-- Assembly -->
   <xacro:chassis
     length="${chassis_length}"
