Commit message: Update extensions and add sensors to urdf

File: src/robot_description/examplo.urdf (robot description, URDF)
Before this commit: robot examplo, 42 links, 41 joints
Links:
- added link lidar_link; collision cylinder length=0.025 radius=0.035; visual cylinder length=0.025 radius=0.035
- added link zed_camera_center; collision box size=0.03 0.12 0.03; visual mesh filename=package://robot_description/meshes/zed2i.stl
- added link zed_left_camera_frame
- added link zed_left_camera_optical_frame
- added link zed_mount_link
- added link zed_right_camera_frame
- added link zed_right_camera_optical_frame
Joints:
- added joint lidar_joint: type fixed, parent chassis_link, child lidar_link, origin xyz=0 -0.045 0.0125 rpy=0 0 0
- added joint zed_camera_center_joint: type fixed, parent zed_mount_link, child zed_camera_center, origin xyz=0 0 0.015 rpy=0 0.0 0
- added joint zed_left_camera_joint: type fixed, parent zed_camera_center, child zed_left_camera_frame, origin xyz=0 0.06 0 rpy=0 0 0
- added joint zed_left_camera_optical_joint: type fixed, parent zed_left_camera_frame, child zed_left_camera_optical_frame, origin xyz=-0.01 0 0 rpy=-1.5707963267948966 0.0 -1.5707963267948966
- added joint zed_mount_joint: type fixed, parent chassis_link, child zed_mount_link, origin xyz=0 0.15 0 rpy=0 0 1.5707963267948966
- added joint zed_right_camera_joint: type fixed, parent zed_camera_center, child zed_right_camera_frame, origin xyz=0 -0.06 0 rpy=0 0 0
- added joint zed_right_camera_optical_joint: type fixed, parent zed_right_camera_frame, child zed_right_camera_optical_frame, origin xyz=-0.01 0 0 rpy=-1.5707963267948966 0.0 -1.5707963267948966

File: src/robot_description/urdf/robots/examplo.urdf.xacro (robot description, xacro)
@@ -7,4 +7,6 @@
   <xacro:include filename="$(find robot_description)/urdf/parts/mecanum_wheel.xacro"/>
   <xacro:include filename="$(find robot_description)/urdf/parts/mecanum_roller.xacro"/>
+  <xacro:include filename="$(find robot_description)/urdf/parts/lidar.xacro"/>
+  <xacro:include filename="$(find robot_description)/urdf/parts/zed_cam.xacro"/>
   <xacro:include filename="$(find robot_description)/urdf/control/drive.xacro"/>
   <!-- Properties -->
@@ -26,4 +28,7 @@
   <xacro:property name="roller_cylinder_radius" value="0.0074" />
   <xacro:property name="roller_length" value="0.0396" />
+  <xacro:property name="lidar_radius" value="0.035" />
+  <xacro:property name="lidar_length" value="0.025" />
+  <xacro:property name="lidar_joint_pos_y" value="-0.045" />
   <!-- Assembly -->
   <xacro:chassis
@@ -77,3 +82,11 @@
     mass="${wheel_weight}"
   />
+  <xacro:lidar
+    radius="${lidar_radius}"
+    length="${lidar_length}"
+    pos_y="${lidar_joint_pos_y}"
+  />
+  <xacro:zed_camera parent="chassis_link">
+    <origin xyz="0 0.15 0" rpy="0 0 ${pi/2}" />
+  </xacro:zed_camera>
 </robot>

Commit message: Update Hardware interface and add depth camera

File: src/robot_description/examplo.urdf (robot description, URDF)
Before this commit: robot examplo, 49 links, 48 joints
Joints:
- joint zed_left_camera_optical_joint: origin xyz=-0.01 0 0 rpy=-1.5707963267948966 0.0 -1.5707963267948966 -> xyz=-0.01 0 0 rpy=-1.5707963267948966 0.0 1.5707963267948966
- joint zed_right_camera_optical_joint: origin xyz=-0.01 0 0 rpy=-1.5707963267948966 0.0 -1.5707963267948966 -> xyz=-0.01 0 0 rpy=-1.5707963267948966 0.0 1.5707963267948966

File: src/robot_description/urdf/parts/zed_cam.xacro (robot description, xacro)
@@ -46,5 +46,5 @@
     <link name="zed_left_camera_optical_frame"/>
     <joint name="zed_left_camera_optical_joint" type="fixed">
-      <origin xyz="${optical_offset_x} 0 0" rpy="-${M_PI/2} 0.0 -${M_PI/2}"/>
+      <origin xyz="${optical_offset_x} 0 0" rpy="-${M_PI/2} 0.0 ${M_PI/2}"/>
       <parent link="zed_left_camera_frame"/>
       <child link="zed_left_camera_optical_frame"/>
@@ -59,5 +59,5 @@
     <link name="zed_right_camera_optical_frame"/>
     <joint name="zed_right_camera_optical_joint" type="fixed">
-      <origin xyz="${optical_offset_x} 0 0" rpy="-${M_PI/2} 0.0 -${M_PI/2}"/>
+      <origin xyz="${optical_offset_x} 0 0" rpy="-${M_PI/2} 0.0 ${M_PI/2}"/>
       <parent link="zed_right_camera_frame"/>
       <child link="zed_right_camera_optical_frame"/>

Commit message: latest cam updates

File: src/robot_description/examplo.urdf (robot description, URDF)
Before this commit: robot examplo, 49 links, 48 joints
Joints:
- joint zed_left_camera_joint: origin xyz=0 0.06 0 rpy=0 0 0 -> xyz=0 0.06 0 rpy=1.5707963267948966 0 -1.5707963267948966
- joint zed_left_camera_optical_joint: origin xyz=-0.01 0 0 rpy=-1.5707963267948966 0.0 1.5707963267948966 -> xyz=-0.01 0 0 rpy=-1.5707963267948966 0.0 -1.5707963267948966
- joint zed_right_camera_optical_joint: origin xyz=-0.01 0 0 rpy=-1.5707963267948966 0.0 1.5707963267948966 -> xyz=-0.01 0 0 rpy=-1.5707963267948966 0.0 -1.5707963267948966

File: src/robot_description/urdf/parts/zed_cam.xacro (robot description, xacro)
@@ -42,9 +42,9 @@
       <parent link="zed_camera_center"/>
       <child link="zed_left_camera_frame"/>
-      <origin xyz="0 ${baseline/2} 0" rpy="0 0 0" />
+      <origin xyz="0 ${baseline/2} 0" rpy="${M_PI/2} 0 -${M_PI/2}" />
     </joint>
     <link name="zed_left_camera_optical_frame"/>
     <joint name="zed_left_camera_optical_joint" type="fixed">
-      <origin xyz="${optical_offset_x} 0 0" rpy="-${M_PI/2} 0.0 ${M_PI/2}"/>
+      <origin xyz="${optical_offset_x} 0 0" rpy="-${M_PI/2} 0.0 -${M_PI/2}"/>
       <parent link="zed_left_camera_frame"/>
       <child link="zed_left_camera_optical_frame"/>
@@ -59,5 +59,5 @@
     <link name="zed_right_camera_optical_frame"/>
     <joint name="zed_right_camera_optical_joint" type="fixed">
-      <origin xyz="${optical_offset_x} 0 0" rpy="-${M_PI/2} 0.0 ${M_PI/2}"/>
+      <origin xyz="${optical_offset_x} 0 0" rpy="-${M_PI/2} 0.0 -${M_PI/2}"/>
       <parent link="zed_right_camera_frame"/>
       <child link="zed_right_camera_optical_frame"/>

Commit message: added meshes

File: src/robot_description/examplo.urdf (robot description, URDF)
Before this commit: robot examplo, 49 links, 48 joints
Links:
- removed link front_left_roller_8
- removed link front_right_roller_8
- removed link rear_left_roller_8
- removed link rear_right_roller_8
- link chassis_link: geometry collision box size=0.18 0.33 0.135; visual mesh filename=package://robot_description/meshes/HillCraterDrivebase.stl scale=0.001 0.001 0.001
- link front_left_mecanum_link: geometry collision cylinder length=0.042 radius=0.030015; visual mesh filename=package://robot_description/meshes/wheel2.stl scale=0.001 0.001 0.001
- link front_left_roller_0: geometry collision sphere radius=0.007485; collision sphere radius=0.007485
- link front_left_roller_1: geometry collision sphere radius=0.007485; collision sphere radius=0.007485
- link front_left_roller_2: geometry collision sphere radius=0.007485; collision sphere radius=0.007485
- link front_left_roller_3: geometry collision sphere radius=0.007485; collision sphere radius=0.007485
- link front_left_roller_4: geometry collision sphere radius=0.007485; collision sphere radius=0.007485
- link front_left_roller_5: geometry collision sphere radius=0.007485; collision sphere radius=0.007485
- link front_left_roller_6: geometry collision sphere radius=0.007485; collision sphere radius=0.007485
- link front_left_roller_7: geometry collision sphere radius=0.007485; collision sphere radius=0.007485
- link front_right_mecanum_link: geometry collision cylinder length=0.042 radius=0.030015; visual mesh filename=package://robot_description/meshes/wheel1.stl scale=0.001 0.001 0.001
- link front_right_roller_0: geometry collision sphere radius=0.007485; collision sphere radius=0.007485
- link front_right_roller_1: geometry collision sphere radius=0.007485; collision sphere radius=0.007485
- link front_right_roller_2: geometry collision sphere radius=0.007485; collision sphere radius=0.007485
- link front_right_roller_3: geometry collision sphere radius=0.007485; collision sphere radius=0.007485
- link front_right_roller_4: geometry collision sphere radius=0.007485; collision sphere radius=0.007485
- link front_right_roller_5: geometry collision sphere radius=0.007485; collision sphere radius=0.007485
- link front_right_roller_6: geometry collision sphere radius=0.007485; collision sphere radius=0.007485
- link front_right_roller_7: geometry collision sphere radius=0.007485; collision sphere radius=0.007485
- link rear_left_mecanum_link: geometry collision cylinder length=0.042 radius=0.030015; visual mesh filename=package://robot_description/meshes/wheel1.stl scale=0.001 0.001 0.001
- link rear_left_roller_0: geometry collision sphere radius=0.007485; collision sphere radius=0.007485
- link rear_left_roller_1: geometry collision sphere radius=0.007485; collision sphere radius=0.007485
- link rear_left_roller_2: geometry collision sphere radius=0.007485; collision sphere radius=0.007485
- link rear_left_roller_3: geometry collision sphere radius=0.007485; collision sphere radius=0.007485
- link rear_left_roller_4: geometry collision sphere radius=0.007485; collision sphere radius=0.007485
- link rear_left_roller_5: geometry collision sphere radius=0.007485; collision sphere radius=0.007485
- link rear_left_roller_6: geometry collision sphere radius=0.007485; collision sphere radius=0.007485
- link rear_left_roller_7: geometry collision sphere radius=0.007485; collision sphere radius=0.007485
- link rear_right_mecanum_link: geometry collision cylinder length=0.042 radius=0.030015; visual mesh filename=package://robot_description/meshes/wheel2.stl scale=0.001 0.001 0.001
- link rear_right_roller_0: geometry collision sphere radius=0.007485; collision sphere radius=0.007485
- link rear_right_roller_1: geometry collision sphere radius=0.007485; collision sphere radius=0.007485
- link rear_right_roller_2: geometry collision sphere radius=0.007485; collision sphere radius=0.007485
- link rear_right_roller_3: geometry collision sphere radius=0.007485; collision sphere radius=0.007485
- link rear_right_roller_4: geometry collision sphere radius=0.007485; collision sphere radius=0.007485
- link rear_right_roller_5: geometry collision sphere radius=0.007485; collision sphere radius=0.007485
- link rear_right_roller_6: geometry collision sphere radius=0.007485; collision sphere radius=0.007485
- link rear_right_roller_7: geometry collision sphere radius=0.007485; collision sphere radius=0.007485
Joints:
- removed joint front_left_roller_8_joint
- removed joint front_right_roller_8_joint
- removed joint rear_left_roller_8_joint
- removed joint rear_right_roller_8_joint
- joint front_left_mecanum_joint: origin xyz=-0.108 0.145 -0.121 rpy=0 1.5707963267948966 0 -> xyz=-0.10075 0.10568 -0.07793 rpy=0 1.5707963267948966 0
- joint front_left_roller_0_joint: origin xyz=0.0 0.0388 0 rpy=-0.0 -0.7853981633974483 0 -> xyz=0.0 0.030015 0 rpy=-0.0 -0.7853981633974483 0
- joint front_left_roller_1_joint: origin xyz=0.024940159255837722 0.02972252439301635 0 rpy=-0.5048442081024438 -0.6016498987064663 0 -> xyz=0.02122381003731422 0.021223810037314224 0 rpy=-0.5553603672697958 -0.5553603672697958 0
- joint front_left_roller_2_joint: origin xyz=0.038210540816873674 0.0067375492934769006 0 rpy=-0.7734662005153561 -0.13638295981692095 0 -> xyz=0.030015 1.8378886838203904e-18 0 rpy=-0.7853981633974483 -4.8091767343044744e-17 0
- joint front_left_roller_3_joint: origin xyz=0.03360178566683622 -0.019399999999999994 0 rpy=-0.6801747615878317 0.392699081698724 0 -> xyz=0.021223810037314224 -0.02122381003731422 0 rpy=-0.5553603672697958 0.5553603672697958 0
- joint front_left_roller_4_joint: origin xyz=0.013270381561035953 -0.03646007368649325 0 rpy=-0.26862199241291235 0.7380328585233872 0 -> xyz=3.675777367640781e-18 -0.030015 0 rpy=-9.618353468608949e-17 0.7853981633974483 0
- joint front_left_roller_5_joint: origin xyz=-0.013270381561035945 -0.03646007368649325 0 rpy=0.2686219924129122 0.7380328585233873 0 -> xyz=-0.02122381003731422 -0.021223810037314227 0 rpy=0.5553603672697958 0.5553603672697959 0
- joint front_left_roller_6_joint: origin xyz=-0.03360178566683621 -0.019400000000000018 0 rpy=0.6801747615878314 0.3926990816987245 0 -> xyz=-0.030015 -5.513666051461171e-18 0 rpy=0.7853981633974483 1.4427530202913423e-16 0
- joint front_left_roller_7_joint: origin xyz=-0.038210540816873674 0.006737549293476883 0 rpy=0.7734662005153561 -0.13638295981692058 0 -> xyz=-0.021223810037314227 0.02122381003731422 0 rpy=0.587317345873812 -0.5013424269205712 0.09416051314509408
- joint front_right_mecanum_joint: origin xyz=0.108 0.145 -0.121 rpy=0 1.5707963267948966 0 -> xyz=0.10075 0.10568 -0.07793 rpy=0 1.5707963267948966 0
- joint front_right_roller_0_joint: origin xyz=0.0 0.0388 0 rpy=0.0 0.7853981633974483 0 -> xyz=0.0 0.030015 0 rpy=0.0 0.7853981633974483 0
- joint front_right_roller_1_joint: origin xyz=0.024940159255837722 0.02972252439301635 0 rpy=0.5048442081024438 0.6016498987064663 0 -> xyz=0.02122381003731422 0.021223810037314224 0 rpy=0.5553603672697958 0.5553603672697958 0
- joint front_right_roller_2_joint: origin xyz=0.038210540816873674 0.0067375492934769006 0 rpy=0.7734662005153561 0.13638295981692095 0 -> xyz=0.030015 1.8378886838203904e-18 0 rpy=0.7853981633974483 4.8091767343044744e-17 0
- joint front_right_roller_3_joint: origin xyz=0.03360178566683622 -0.019399999999999994 0 rpy=0.6801747615878317 -0.392699081698724 0 -> xyz=0.021223810037314224 -0.02122381003731422 0 rpy=0.5553603672697958 -0.5553603672697958 0
- joint front_right_roller_4_joint: origin xyz=0.013270381561035953 -0.03646007368649325 0 rpy=0.26862199241291235 -0.7380328585233872 0 -> xyz=3.675777367640781e-18 -0.030015 0 rpy=9.618353468608949e-17 -0.7853981633974483 0
- joint front_right_roller_5_joint: origin xyz=-0.013270381561035945 -0.03646007368649325 0 rpy=-0.2686219924129122 -0.7380328585233873 0 -> xyz=-0.02122381003731422 -0.021223810037314227 0 rpy=-0.5553603672697958 -0.5553603672697959 0
- joint front_right_roller_6_joint: origin xyz=-0.03360178566683621 -0.019400000000000018 0 rpy=-0.6801747615878314 -0.3926990816987245 0 -> xyz=-0.030015 -5.513666051461171e-18 0 rpy=-0.7853981633974483 -1.4427530202913423e-16 0
- joint front_right_roller_7_joint: origin xyz=-0.038210540816873674 0.006737549293476883 0 rpy=-0.7734662005153561 0.13638295981692058 0 -> xyz=-0.021223810037314227 0.02122381003731422 0 rpy=-0.5234033886657797 0.6093783076190201 0.09416051314509408
- joint rear_left_mecanum_joint: origin xyz=-0.108 -0.145 -0.121 rpy=0 -1.5707963267948966 0 -> xyz=-0.10075 -0.10568 -0.07793 rpy=0 -1.5707963267948966 0
- joint rear_left_roller_0_joint: origin xyz=0.0 0.0388 0 rpy=0.0 0.7853981633974483 0 -> xyz=0.0 0.030015 0 rpy=0.0 0.7853981633974483 0
- joint rear_left_roller_1_joint: origin xyz=0.024940159255837722 0.02972252439301635 0 rpy=0.5048442081024438 0.6016498987064663 0 -> xyz=0.02122381003731422 0.021223810037314224 0 rpy=0.5553603672697958 0.5553603672697958 0
- joint rear_left_roller_2_joint: origin xyz=0.038210540816873674 0.0067375492934769006 0 rpy=0.7734662005153561 0.13638295981692095 0 -> xyz=0.030015 1.8378886838203904e-18 0 rpy=0.7853981633974483 4.8091767343044744e-17 0
- joint rear_left_roller_3_joint: origin xyz=0.03360178566683622 -0.019399999999999994 0 rpy=0.6801747615878317 -0.392699081698724 0 -> xyz=0.021223810037314224 -0.02122381003731422 0 rpy=0.5553603672697958 -0.5553603672697958 0
- joint rear_left_roller_4_joint: origin xyz=0.013270381561035953 -0.03646007368649325 0 rpy=0.26862199241291235 -0.7380328585233872 0 -> xyz=3.675777367640781e-18 -0.030015 0 rpy=9.618353468608949e-17 -0.7853981633974483 0
- joint rear_left_roller_5_joint: origin xyz=-0.013270381561035945 -0.03646007368649325 0 rpy=-0.2686219924129122 -0.7380328585233873 0 -> xyz=-0.02122381003731422 -0.021223810037314227 0 rpy=-0.5553603672697958 -0.5553603672697959 0
- joint rear_left_roller_6_joint: origin xyz=-0.03360178566683621 -0.019400000000000018 0 rpy=-0.6801747615878314 -0.3926990816987245 0 -> xyz=-0.030015 -5.513666051461171e-18 0 rpy=-0.7853981633974483 -1.4427530202913423e-16 0
- joint rear_left_roller_7_joint: origin xyz=-0.038210540816873674 0.006737549293476883 0 rpy=-0.7734662005153561 0.13638295981692058 0 -> xyz=-0.021223810037314227 0.02122381003731422 0 rpy=-0.5234033886657797 0.6093783076190201 0.09416051314509408
- joint rear_right_mecanum_joint: origin xyz=0.108 -0.145 -0.121 rpy=0 -1.5707963267948966 0 -> xyz=0.10075 -0.10568 -0.07793 rpy=0 -1.5707963267948966 0
- joint rear_right_roller_0_joint: origin xyz=0.0 0.0388 0 rpy=-0.0 -0.7853981633974483 0 -> xyz=0.0 0.030015 0 rpy=-0.0 -0.7853981633974483 0
- joint rear_right_roller_1_joint: origin xyz=0.024940159255837722 0.02972252439301635 0 rpy=-0.5048442081024438 -0.6016498987064663 0 -> xyz=0.02122381003731422 0.021223810037314224 0 rpy=-0.5553603672697958 -0.5553603672697958 0
- joint rear_right_roller_2_joint: origin xyz=0.038210540816873674 0.0067375492934769006 0 rpy=-0.7734662005153561 -0.13638295981692095 0 -> xyz=0.030015 1.8378886838203904e-18 0 rpy=-0.7853981633974483 -4.8091767343044744e-17 0
- joint rear_right_roller_3_joint: origin xyz=0.03360178566683622 -0.019399999999999994 0 rpy=-0.6801747615878317 0.392699081698724 0 -> xyz=0.021223810037314224 -0.02122381003731422 0 rpy=-0.5553603672697958 0.5553603672697958 0
- joint rear_right_roller_4_joint: origin xyz=0.013270381561035953 -0.03646007368649325 0 rpy=-0.26862199241291235 0.7380328585233872 0 -> xyz=3.675777367640781e-18 -0.030015 0 rpy=-9.618353468608949e-17 0.7853981633974483 0
- joint rear_right_roller_5_joint: origin xyz=-0.013270381561035945 -0.03646007368649325 0 rpy=0.2686219924129122 0.7380328585233873 0 -> xyz=-0.02122381003731422 -0.021223810037314227 0 rpy=0.5553603672697958 0.5553603672697959 0
- joint rear_right_roller_6_joint: origin xyz=-0.03360178566683621 -0.019400000000000018 0 rpy=0.6801747615878314 0.3926990816987245 0 -> xyz=-0.030015 -5.513666051461171e-18 0 rpy=0.7853981633974483 1.4427530202913423e-16 0
- joint rear_right_roller_7_joint: origin xyz=-0.038210540816873674 0.006737549293476883 0 rpy=0.7734662005153561 -0.13638295981692058 0 -> xyz=-0.021223810037314227 0.02122381003731422 0 rpy=0.587317345873812 -0.5013424269205712 0.09416051314509408

File: src/robot_description/urdf/parts/chassis.xacro (robot description, xacro)
@@ -10,5 +10,5 @@
         <origin xyz="0 0 0" rpy="0 0 0"/>
         <geometry>
-          <mesh filename="package://robot_description/meshes/chassis.stl" scale="0.001 0.001 0.001"/>
+          <mesh filename="package://robot_description/meshes/HillCraterDrivebase.stl" scale="0.001 0.001 0.001"/>
         </geometry>
         <material name="blue"/>

File: src/robot_description/urdf/parts/mecanum_roller.xacro (robot description, xacro)
@@ -5,5 +5,5 @@
     <xacro:property name="type_offset" value="${(type * 2 - 3) * -1}" />
     <!-- Compute incremental radians to place the roller around the hub -->
-    <xacro:property name="roller_radians" value="${2 * pi / roller_total * number}" />
+    <xacro:property name="roller_radians" value="${(2 * pi / roller_total * number)}" />
     <!-- Figure out the x and y position of the roller from radian value -->
     <xacro:property name="roller_x_pos" value="${sin(roller_radians) * wheel_radius}" />
@@ -12,9 +12,21 @@
     <xacro:property name="roller_x_rot" value="${sin(roller_radians) * (pi/4) * type_offset}" />
     <xacro:property name="roller_y_rot" value="${cos(roller_radians) * (pi/4) * type_offset}" />
+    <xacro:property name="roller_z_rot" value="0"/>
+    <xacro:if value="${number==1}">
+    </xacro:if>
+    <xacro:if value="${number==3}">
+    </xacro:if>
+    <xacro:if value="${number==5}">
+    </xacro:if>
+    <xacro:if value="${number==7}">
+      <xacro:property name="roller_x_rot" value="${(sin(roller_radians) * (pi/4) * type_offset)+(1.831*pi/180)}" />
+      <xacro:property name="roller_y_rot" value="${(cos(roller_radians) * (pi/4) * type_offset)+(3.095*pi/180)}" />
+      <xacro:property name="roller_z_rot" value="${(5.395*pi/180)}"/>
+    </xacro:if>
     <link name="${name}_roller_${number}">
       <visual>
         <origin xyz="0 0 0" rpy="0 0 0"/>
         <geometry>
-          <mesh filename="package://robot_description/meshes/roller.stl" scale="0.001 0.001 0.001"/>
+          <mesh filename="package://robot_description/meshes/rolle2r.stl" scale="0.001 0.001 0.001"/>
         </geometry>
         <material name="grey"/>
@@ -52,5 +64,5 @@
     </link>
     <joint name="${name}_roller_${number}_joint" type="continuous">
-      <origin xyz="${roller_x_pos} ${roller_y_pos} 0" rpy="${roller_x_rot} ${roller_y_rot} 0"/>
+      <origin xyz="${roller_x_pos} ${roller_y_pos} 0" rpy="${roller_x_rot} ${roller_y_rot} ${roller_z_rot}"/>
       <parent link="${name}_mecanum_link"/>
       <child link="${name}_roller_${number}"/>

File: src/robot_description/urdf/parts/mecanum_wheel.xacro (robot description, xacro)
@@ -9,5 +9,5 @@
         <origin xyz="0 0 0" rpy="0 0 0"/>
         <geometry>
-          <mesh filename="package://robot_description/meshes/mec_hub_${type}.stl" scale="0.001 0.001 0.001"/>
+          <mesh filename="package://robot_description/meshes/wheel${type}.stl" scale="0.001 0.001 0.001"/>
         </geometry>
         <material name="orange"/>
@@ -26,5 +26,5 @@
       <axis xyz="0.0 0.0 ${copysign(1, (flip * -1))}"/>
     </joint>
-    <!-- There will be 9 rollers for each wheel -->
+    <!-- There will be 8 rollers for each wheel -->
     <xacro:roller name="${name}" number="0" />
     <xacro:roller name="${name}" number="1" />
@@ -35,5 +35,4 @@
     <xacro:roller name="${name}" number="6" />
     <xacro:roller name="${name}" number="7" />
-    <xacro:roller name="${name}" number="8" />
   </xacro:macro>
 </robot>

File: src/robot_description/urdf/robots/examplo.urdf.xacro (robot description, xacro)
@@ -15,12 +15,12 @@
   <xacro:property name="chassis_height" value="0.135" />
   <xacro:property name="chassis_weight" value="2.45" />
-  <xacro:property name="wheel_radius" value="${0.0194/2 + 0.0291}" />
+  <xacro:property name="wheel_radius" value="${0.0375-0.01497/2}" />
   <xacro:property name="wheel_thickness" value="0.042" />
   <xacro:property name="wheel_weight" value="0.136" />
-  <xacro:property name="wheel_offset" value="${wheel_thickness/2 - 0.003}" />
-  <xacro:property name="wheel_joint_pos_x" value="0.09" />
-  <xacro:property name="wheel_joint_pos_y" value="0.145" />
-  <xacro:property name="wheel_joint_pos_z" value="0.121" />
-  <xacro:property name="roller_total" value="9" />
+  <xacro:property name="wheel_offset" value="0" />
+  <xacro:property name="wheel_joint_pos_x" value="0.10075" />
+  <xacro:property name="wheel_joint_pos_y" value="0.10568" />
+  <xacro:property name="wheel_joint_pos_z" value="0.07793" />
+  <xacro:property name="roller_total" value="8" />
   <xacro:property name="roller_middle_radius" value="${0.01621/2}" />
   <xacro:property name="roller_second_radius" value="${0.01591/2}" />
