Commit message: updated physics

File: src/robot_description/examplo.urdf (robot description, URDF)
Before this commit: robot examplo, 45 links, 44 joints
Links:
- link chassis_link: geometry collision box size=0.18 0.33 0.0675; visual mesh filename=package://robot_description/meshes/HillCraterDrivebase.stl scale=0.001 0.001 0.001
- link front_left_mecanum_link: mass 0.136 -> 1.1360000000000001
- link front_left_roller_0: mass None -> 0.07; geometry collision mesh filename=package://robot_description/meshes/rolle2r.stl scale=0.001 0.001 0.001; visual mesh filename=package://robot_description/meshes/rolle2r.stl scale=0.001 0.001 0.001
- link front_left_roller_1: mass None -> 0.07; geometry collision mesh filename=package://robot_description/meshes/rolle2r.stl scale=0.001 0.001 0.001; visual mesh filename=package://robot_description/meshes/rolle2r.stl scale=0.001 0.001 0.001
- link front_left_roller_2: mass None -> 0.07; geometry collision mesh filename=package://robot_description/meshes/rolle2r.stl scale=0.001 0.001 0.001; visual mesh filename=package://robot_description/meshes/rolle2r.stl scale=0.001 0.001 0.001
- link front_left_roller_3: mass None -> 0.07; geometry collision mesh filename=package://robot_description/meshes/rolle2r.stl scale=0.001 0.001 0.001; visual mesh filename=package://robot_description/meshes/rolle2r.stl scale=0.001 0.001 0.001
- link front_left_roller_4: mass None -> 0.07; geometry collision mesh filename=package://robot_description/meshes/rolle2r.stl scale=0.001 0.001 0.001; visual mesh filename=package://robot_description/meshes/rolle2r.stl scale=0.001 0.001 0.001
- link front_left_roller_5: mass None -> 0.07; geometry collision mesh filename=package://robot_description/meshes/rolle2r.stl scale=0.001 0.001 0.001; visual mesh filename=package://robot_description/meshes/rolle2r.stl scale=0.001 0.001 0.001
- link front_left_roller_6: mass None -> 0.07; geometry collision mesh filename=package://robot_description/meshes/rolle2r.stl scale=0.001 0.001 0.001; visual mesh filename=package://robot_description/meshes/rolle2r.stl scale=0.001 0.001 0.001
- link front_left_roller_7: mass None -> 0.07; geometry collision mesh filename=package://robot_description/meshes/rolle2r.stl scale=0.001 0.001 0.001; visual mesh filename=package://robot_description/meshes/rolle2r.stl scale=0.001 0.001 0.001
- link front_right_mecanum_link: mass 0.136 -> 1.1360000000000001
- link front_right_roller_0: mass None -> 0.07; geometry collision mesh filename=package://robot_description/meshes/rolle2r.stl scale=0.001 0.001 0.001; visual mesh filename=package://robot_description/meshes/rolle2r.stl scale=0.001 0.001 0.001
- link front_right_roller_1: mass None -> 0.07; geometry collision mesh filename=package://robot_description/meshes/rolle2r.stl scale=0.001 0.001 0.001; visual mesh filename=package://robot_description/meshes/rolle2r.stl scale=0.001 0.001 0.001
- link front_right_roller_2: mass None -> 0.07; geometry collision mesh filename=package://robot_description/meshes/rolle2r.stl scale=0.001 0.001 0.001; visual mesh filename=package://robot_description/meshes/rolle2r.stl scale=0.001 0.001 0.001
- link front_right_roller_3: mass None -> 0.07; geometry collision mesh filename=package://robot_description/meshes/rolle2r.stl scale=0.001 0.001 0.001; visual mesh filename=package://robot_description/meshes/rolle2r.stl scale=0.001 0.001 0.001
- link front_right_roller_4: mass None -> 0.07; geometry collision mesh filename=package://robot_description/meshes/rolle2r.stl scale=0.001 0.001 0.001; visual mesh filename=package://robot_description/meshes/rolle2r.stl scale=0.001 0.001 0.001
- link front_right_roller_5: mass None -> 0.07; geometry collision mesh filename=package://robot_description/meshes/rolle2r.stl scale=0.001 0.001 0.001; visual mesh filename=package://robot_description/meshes/rolle2r.stl scale=0.001 0.001 0.001
- link front_right_roller_6: mass None -> 0.07; geometry collision mesh filename=package://robot_description/meshes/rolle2r.stl scale=0.001 0.001 0.001; visual mesh filename=package://robot_description/meshes/rolle2r.stl scale=0.001 0.001 0.001
- link front_right_roller_7: mass None -> 0.07; geometry collision mesh filename=package://robot_description/meshes/rolle2r.stl scale=0.001 0.001 0.001; visual mesh filename=package://robot_description/meshes/rolle2r.stl scale=0.001 0.001 0.001
- link rear_left_mecanum_link: mass 0.136 -> 1.1360000000000001
- link rear_left_roller_0: mass None -> 0.07; geometry collision mesh filename=package://robot_description/meshes/rolle2r.stl scale=0.001 0.001 0.001; visual mesh filename=package://robot_description/meshes/rolle2r.stl scale=0.001 0.001 0.001
- link rear_left_roller_1: mass None -> 0.07; geometry collision mesh filename=package://robot_description/meshes/rolle2r.stl scale=0.001 0.001 0.001; visual mesh filename=package://robot_description/meshes/rolle2r.stl scale=0.001 0.001 0.001
- link rear_left_roller_2: mass None -> 0.07; geometry collision mesh filename=package://robot_description/meshes/rolle2r.stl scale=0.001 0.001 0.001; visual mesh filename=package://robot_description/meshes/rolle2r.stl scale=0.001 0.001 0.001
- link rear_left_roller_3: mass None -> 0.07; geometry collision mesh filename=package://robot_description/meshes/rolle2r.stl scale=0.001 0.001 0.001; visual mesh filename=package://robot_description/meshes/rolle2r.stl scale=0.001 0.001 0.001
- link rear_left_roller_4: mass None -> 0.07; geometry collision mesh filename=package://robot_description/meshes/rolle2r.stl scale=0.001 0.001 0.001; visual mesh filename=package://robot_description/meshes/rolle2r.stl scale=0.001 0.001 0.001
- link rear_left_roller_5: mass None -> 0.07; geometry collision mesh filename=package://robot_description/meshes/rolle2r.stl scale=0.001 0.001 0.001; visual mesh filename=package://robot_description/meshes/rolle2r.stl scale=0.001 0.001 0.001
- link rear_left_roller_6: mass None -> 0.07; geometry collision mesh filename=package://robot_description/meshes/rolle2r.stl scale=0.001 0.001 0.001; visual mesh filename=package://robot_description/meshes/rolle2r.stl scale=0.001 0.001 0.001
- link rear_left_roller_7: mass None -> 0.07; geometry collision mesh filename=package://robot_description/meshes/rolle2r.stl scale=0.001 0.001 0.001; visual mesh filename=package://robot_description/meshes/rolle2r.stl scale=0.001 0.001 0.001
- link rear_right_mecanum_link: mass 0.136 -> 1.1360000000000001
- link rear_right_roller_0: mass None -> 0.07; geometry collision mesh filename=package://robot_description/meshes/rolle2r.stl scale=0.001 0.001 0.001; visual mesh filename=package://robot_description/meshes/rolle2r.stl scale=0.001 0.001 0.001
- link rear_right_roller_1: mass None -> 0.07; geometry collision mesh filename=package://robot_description/meshes/rolle2r.stl scale=0.001 0.001 0.001; visual mesh filename=package://robot_description/meshes/rolle2r.stl scale=0.001 0.001 0.001
- link rear_right_roller_2: mass None -> 0.07; geometry collision mesh filename=package://robot_description/meshes/rolle2r.stl scale=0.001 0.001 0.001; visual mesh filename=package://robot_description/meshes/rolle2r.stl scale=0.001 0.001 0.001
- link rear_right_roller_3: mass None -> 0.07; geometry collision mesh filename=package://robot_description/meshes/rolle2r.stl scale=0.001 0.001 0.001; visual mesh filename=package://robot_description/meshes/rolle2r.stl scale=0.001 0.001 0.001
- link rear_right_roller_4: mass None -> 0.07; geometry collision mesh filename=package://robot_description/meshes/rolle2r.stl scale=0.001 0.001 0.001; visual mesh filename=package://robot_description/meshes/rolle2r.stl scale=0.001 0.001 0.001
- link rear_right_roller_5: mass None -> 0.07; geometry collision mesh filename=package://robot_description/meshes/rolle2r.stl scale=0.001 0.001 0.001; visual mesh filename=package://robot_description/meshes/rolle2r.stl scale=0.001 0.001 0.001
- link rear_right_roller_6: mass None -> 0.07; geometry collision mesh filename=package://robot_description/meshes/rolle2r.stl scale=0.001 0.001 0.001; visual mesh filename=package://robot_description/meshes/rolle2r.stl scale=0.001 0.001 0.001
- link rear_right_roller_7: mass None -> 0.07; geometry collision mesh filename=package://robot_description/meshes/rolle2r.stl scale=0.001 0.001 0.001; visual mesh filename=package://robot_description/meshes/rolle2r.stl scale=0.001 0.001 0.001

File: src/robot_description/urdf/parts/chassis.xacro (robot description, xacro)
@@ -15,7 +15,7 @@
       </visual>
       <collision>
-        <origin xyz="0 0 -${height / 2}" rpy="0 0 0"/>
+        <origin xyz="0 0 0" rpy="0 0 0"/>
         <geometry>
-          <box size="${length} ${width} ${height}"/>
+          <box size="${length} ${width} ${height/2}"/>
         </geometry>
       </collision>

File: src/robot_description/urdf/parts/mecanum_roller.xacro (robot description, xacro)
@@ -32,5 +32,5 @@
         <material name="grey"/>
       </visual>
-      <collision>
+      <!-- <collision>
         <origin xyz="0 0 0" rpy="0 0 0"/>
         <geometry>
@@ -61,5 +61,14 @@
           <sphere radius="${roller_third_radius}"/>
         </geometry>
+      </collision> -->
+      <collision>
+        <origin xyz="0 0 0" rpy="0 0 0"/>
+        <geometry>
+          <mesh filename="package://robot_description/meshes/rolle2r.stl" scale="0.001 0.001 0.001"/>
+        </geometry>
       </collision>
+      <xacro:inertial_cylinder mass="0.07" radius="${roller_cylinder_radius}" length="${roller_length}">
+        <origin xyz="0 0 0" rpy="0 0 0"/>
+      </xacro:inertial_cylinder>
     </link>
     <joint name="${name}_roller_${number}_joint" type="continuous">

File: src/robot_description/urdf/parts/mecanum_wheel.xacro (robot description, xacro)
@@ -3,5 +3,5 @@
   <xacro:macro name="mecanum_with_rollers" params="name type radius width flip pos_x pos_y pos_z mass">
     <link name="${name}_mecanum_link">
-      <xacro:inertial_cylinder mass="${mass}" length="${width}" radius="${radius}">
+      <xacro:inertial_cylinder mass="${mass+1}" length="${width}" radius="${radius}">
         <origin xyz="0 0 0" rpy="0 ${pi/2} 0"/>
       </xacro:inertial_cylinder>
