Commit message: added submechanisms/ simplified meshes

File: src/robot_description/examplo.urdf (robot description, URDF)
Before this commit: robot examplo, 45 links, 44 joints
Links:
- removed link lidar_link
- removed link zed_camera_center
- removed link zed_left_camera_frame
- removed link zed_left_camera_optical_frame
- removed link zed_mount_link
- removed link zed_right_camera_frame
- removed link zed_right_camera_optical_frame
- added link bridge_holder_link, mass 0.135; collision box size=0.135 0.18 0.165; visual mesh filename=package://robot_description/meshes/bridge_holder.stl scale=0.001 0.001 0.001
- added link bridge_latch_link, mass 0.135; collision box size=2.45 0.18 0.165; visual mesh filename=package://robot_description/meshes/bridge_latch.stl scale=0.001 0.001 0.001
- added link camera_1_link, mass 2.45; collision box size=0.18 0.33 0.0675; visual mesh filename=package://robot_description/meshes/camera.stl scale=0.001 0.001 0.001
- added link camera_2_link, mass 2.45; collision box size=0.18 0.33 0.0675; visual mesh filename=package://robot_description/meshes/camera.stl scale=0.001 0.001 0.001
- added link camera_stand_link, mass 2.45; collision box size=0.18 0.33 0.0675; visual mesh filename=package://robot_description/meshes/camera_stand.stl scale=0.001 0.001 0.001
- added link color_sensor_link, mass 2.45; collision box size=0.18 0.33 0.0675; visual mesh filename=package://robot_description/meshes/color_sensor.stl scale=0.001 0.001 0.001
- added link grr_brain_link, mass 2.45; collision box size=0.18 0.33 0.0675; visual mesh filename=package://robot_description/meshes/brain.stl scale=0.001 0.001 0.001
- added link small_package_grabber_link, mass 2.45; collision box size=0.18 0.33 0.0675; visual mesh filename=package://robot_description/meshes/small_package_grabber.stl scale=0.001 0.001 0.001
- added link small_package_grabber_roller_1_link, mass 2.45; collision cylinder length=0.33 radius=0.18; visual mesh filename=package://robot_description/meshes/small_package_grabber_ro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 scale=0.001 0.001 0.001
- added link small_package_grabber_roller_2_link, mass 2.45; collision cylinder length=0.33 radius=0.18; visual mesh filename=package://robot_description/meshes/small_package_grabber_ro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 scale=0.001 0.001 0.001
- added link small_package_grabber_roller_3_link, mass 2.45; collision cylinder length=0.33 radius=0.18; visual mesh filename=package://robot_description/meshes/small_package_grabber_ro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 scale=0.001 0.001 0.001
- added link small_package_grabber_roller_4_link, mass 2.45; collision cylinder length=0.33 radius=0.18; visual mesh filename=package://robot_description/meshes/small_package_grabber_ro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 scale=0.001 0.001 0.001
- added link small_package_sweeper_link, mass 2.45; collision cylinder length=0.135 radius=0.18; visual mesh filename=package://robot_description/meshes/small_package_sweeper.stl scale=0.001 0.001 0.001
- added link small_package_sweeper_roller_link, mass 2.45; collision cylinder length=0.135 radius=0.18; visual mesh filename=package://robot_description/meshes/small_package_sweeper_ro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 scale=0.001 0.001 0.001
- added link small_package_sweeper_servo_link, mass 2.45; collision box size=0.18 0.33 0.0675; visual mesh filename=package://robot_description/meshes/small_package_sweeper_se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 scale=0.001 0.001 0.001
- link chassis_link: geometry collision box size=0.18 0.33 0.0675; visual mesh filename=package://robot_description/meshes/slim_drivebase.stl scale=0.001 0.001 0.001
- link front_left_mecanum_link: geometry collision cylinder length=0.042 radius=0.030015; visual mesh filename=package://robot_description/meshes/mechanum_wheel_2.stl scale=0.001 0.001 0.001
- link front_left_roller_0: geometry collision mesh filename=package://robot_description/meshes/mechanum_roller.stl scale=0.001 0.001 0.001; visual mesh filename=package://robot_description/meshes/mechanum_roller.stl scale=0.001 0.001 0.001
- link front_left_roller_1: geometry collision mesh filename=package://robot_description/meshes/mechanum_roller.stl scale=0.001 0.001 0.001; visual mesh filename=package://robot_description/meshes/mechanum_roller.stl scale=0.001 0.001 0.001
- link front_left_roller_2: geometry collision mesh filename=package://robot_description/meshes/mechanum_roller.stl scale=0.001 0.001 0.001; visual mesh filename=package://robot_description/meshes/mechanum_roller.stl scale=0.001 0.001 0.001
- link front_left_roller_3: geometry collision mesh filename=package://robot_description/meshes/mechanum_roller.stl scale=0.001 0.001 0.001; visual mesh filename=package://robot_description/meshes/mechanum_roller.stl scale=0.001 0.001 0.001
- link front_left_roller_4: geometry collision mesh filename=package://robot_description/meshes/mechanum_roller.stl scale=0.001 0.001 0.001; visual mesh filename=package://robot_description/meshes/mechanum_roller.stl scale=0.001 0.001 0.001
- link front_left_roller_5: geometry collision mesh filename=package://robot_description/meshes/mechanum_roller.stl scale=0.001 0.001 0.001; visual mesh filename=package://robot_description/meshes/mechanum_roller.stl scale=0.001 0.001 0.001
- link front_left_roller_6: geometry collision mesh filename=package://robot_description/meshes/mechanum_roller.stl scale=0.001 0.001 0.001; visual mesh filename=package://robot_description/meshes/mechanum_roller.stl scale=0.001 0.001 0.001
- link front_left_roller_7: geometry collision mesh filename=package://robot_description/meshes/mechanum_roller.stl scale=0.001 0.001 0.001; visual mesh filename=package://robot_description/meshes/mechanum_roller.stl scale=0.001 0.001 0.001
- link front_right_mecanum_link: geometry collision cylinder length=0.042 radius=0.030015; visual mesh filename=package://robot_description/meshes/mechanum_wheel_1.stl scale=0.001 0.001 0.001
- link front_right_roller_0: geometry collision mesh filename=package://robot_description/meshes/mechanum_roller.stl scale=0.001 0.001 0.001; visual mesh filename=package://robot_description/meshes/mechanum_roller.stl scale=0.001 0.001 0.001
- link front_right_roller_1: geometry collision mesh filename=package://robot_description/meshes/mechanum_roller.stl scale=0.001 0.001 0.001; visual mesh filename=package://robot_description/meshes/mechanum_roller.stl scale=0.001 0.001 0.001
- link front_right_roller_2: geometry collision mesh filename=package://robot_description/meshes/mechanum_roller.stl scale=0.001 0.001 0.001; visual mesh filename=package://robot_description/meshes/mechanum_roller.stl scale=0.001 0.001 0.001
- link front_right_roller_3: geometry collision mesh filename=package://robot_description/meshes/mechanum_roller.stl scale=0.001 0.001 0.001; visual mesh filename=package://robot_description/meshes/mechanum_roller.stl scale=0.001 0.001 0.001
- link front_right_roller_4: geometry collision mesh filename=package://robot_description/meshes/mechanum_roller.stl scale=0.001 0.001 0.001; visual mesh filename=package://robot_description/meshes/mechanum_roller.stl scale=0.001 0.001 0.001
- link front_right_roller_5: geometry collision mesh filename=package://robot_description/meshes/mechanum_roller.stl scale=0.001 0.001 0.001; visual mesh filename=package://robot_description/meshes/mechanum_roller.stl scale=0.001 0.001 0.001
- link front_right_roller_6: geometry collision mesh filename=package://robot_description/meshes/mechanum_roller.stl scale=0.001 0.001 0.001; visual mesh filename=package://robot_description/meshes/mechanum_roller.stl scale=0.001 0.001 0.001
- link front_right_roller_7: geometry collision mesh filename=package://robot_description/meshes/mechanum_roller.stl scale=0.001 0.001 0.001; visual mesh filename=package://robot_description/meshes/mechanum_roller.stl scale=0.001 0.001 0.001
- link rear_left_mecanum_link: geometry collision cylinder length=0.042 radius=0.030015; visual mesh filename=package://robot_description/meshes/mechanum_wheel_1.stl scale=0.001 0.001 0.001
- link rear_left_roller_0: geometry collision mesh filename=package://robot_description/meshes/mechanum_roller.stl scale=0.001 0.001 0.001; visual mesh filename=package://robot_description/meshes/mechanum_roller.stl scale=0.001 0.001 0.001
- link rear_left_roller_1: geometry collision mesh filename=package://robot_description/meshes/mechanum_roller.stl scale=0.001 0.001 0.001; visual mesh filename=package://robot_description/meshes/mechanum_roller.stl scale=0.001 0.001 0.001
- link rear_left_roller_2: geometry collision mesh filename=package://robot_description/meshes/mechanum_roller.stl scale=0.001 0.001 0.001; visual mesh filename=package://robot_description/meshes/mechanum_roller.stl scale=0.001 0.001 0.001
- link rear_left_roller_3: geometry collision mesh filename=package://robot_description/meshes/mechanum_roller.stl scale=0.001 0.001 0.001; visual mesh filename=package://robot_description/meshes/mechanum_roller.stl scale=0.001 0.001 0.001
- link rear_left_roller_4: geometry collision mesh filename=package://robot_description/meshes/mechanum_roller.stl scale=0.001 0.001 0.001; visual mesh filename=package://robot_description/meshes/mechanum_roller.stl scale=0.001 0.001 0.001
- link rear_left_roller_5: geometry collision mesh filename=package://robot_description/meshes/mechanum_roller.stl scale=0.001 0.001 0.001; visual mesh filename=package://robot_description/meshes/mechanum_roller.stl scale=0.001 0.001 0.001
- link rear_left_roller_6: geometry collision mesh filename=package://robot_description/meshes/mechanum_roller.stl scale=0.001 0.001 0.001; visual mesh filename=package://robot_description/meshes/mechanum_roller.stl scale=0.001 0.001 0.001
- link rear_left_roller_7: geometry collision mesh filename=package://robot_description/meshes/mechanum_roller.stl scale=0.001 0.001 0.001; visual mesh filename=package://robot_description/meshes/mechanum_roller.stl scale=0.001 0.001 0.001
- link rear_right_mecanum_link: geometry collision cylinder length=0.042 radius=0.030015; visual mesh filename=package://robot_description/meshes/mechanum_wheel_2.stl scale=0.001 0.001 0.001
- link rear_right_roller_0: geometry collision mesh filename=package://robot_description/meshes/mechanum_roller.stl scale=0.001 0.001 0.001; visual mesh filename=package://robot_description/meshes/mechanum_roller.stl scale=0.001 0.001 0.001
- link rear_right_roller_1: geometry collision mesh filename=package://robot_description/meshes/mechanum_roller.stl scale=0.001 0.001 0.001; visual mesh filename=package://robot_description/meshes/mechanum_roller.stl scale=0.001 0.001 0.001
- link rear_right_roller_2: geometry collision mesh filename=package://robot_description/meshes/mechanum_roller.stl scale=0.001 0.001 0.001; visual mesh filename=package://robot_description/meshes/mechanum_roller.stl scale=0.001 0.001 0.001
- link rear_right_roller_3: geometry collision mesh filename=package://robot_description/meshes/mechanum_roller.stl scale=0.001 0.001 0.001; visual mesh filename=package://robot_description/meshes/mechanum_roller.stl scale=0.001 0.001 0.001
- link rear_right_roller_4: geometry collision mesh filename=package://robot_description/meshes/mechanum_roller.stl scale=0.001 0.001 0.001; visual mesh filename=package://robot_description/meshes/mechanum_roller.stl scale=0.001 0.001 0.001
- link rear_right_roller_5: geometry collision mesh filename=package://robot_description/meshes/mechanum_roller.stl scale=0.001 0.001 0.001; visual mesh filename=package://robot_description/meshes/mechanum_roller.stl scale=0.001 0.001 0.001
- link rear_right_roller_6: geometry collision mesh filename=package://robot_description/meshes/mechanum_roller.stl scale=0.001 0.001 0.001; visual mesh filename=package://robot_description/meshes/mechanum_roller.stl scale=0.001 0.001 0.001
- link rear_right_roller_7: geometry collision mesh filename=package://robot_description/meshes/mechanum_roller.stl scale=0.001 0.001 0.001; visual mesh filename=package://robot_description/meshes/mechanum_roller.stl scale=0.001 0.001 0.001
Joints:
- removed joint lidar_joint
- removed joint zed_camera_center_joint
- removed joint zed_left_camera_joint
- removed joint zed_left_camera_optical_joint
- removed joint zed_mount_joint
- removed joint zed_right_camera_joint
- removed joint zed_right_camera_optical_joint
- added joint bridge_holder_joint: type fixed, parent chassis_link, child bridge_holder_link, origin xyz=0.0 -0.04 0.03 rpy=0 0 0
- added joint bridge_latch_joint: type fixed, parent camera_stand_link, child bridge_latch_link, origin xyz=0.0 0.0 0.0 rpy=0 0 0
- added joint camera_1_joint: type fixed, parent camera_stand_link, child camera_1_link, origin xyz=0.02 -0.05 0.09 rpy=0 0 0
- added joint camera_2_joint: type fixed, parent camera_stand_link, child camera_2_link, origin xyz=0.045 0.04 0.07 rpy=0 0 0
- added joint camera_stand_joint: type fixed, parent chassis_link, child camera_stand_link, origin xyz=0.0 -0.08 0.145
- added joint color_sensor_joint: type fixed, parent bridge_holder_link, child color_sensor_link, origin xyz=0.0 -0.11 0.04 rpy=0 0 0
- added joint grr_brain_joint: type fixed, parent chassis_link, child grr_brain_link, origin xyz=-0.09 -0.14 0.07
- added joint small_package_grabber_joint: type fixed, parent chassis_link, child small_package_grabber_link, origin xyz=-0.03 0.1 0.03
- added joint small_package_grabber_roller_1_joint: type continuous, parent small_package_grabber_link, child small_package_grabber_roller_1_link, origin xyz=0.035 0.03 -0.04 rpy=0 0 0, axis 1 0 0
- added joint small_package_grabber_roller_2_joint: type continuous, parent small_package_grabber_link, child small_package_grabber_roller_2_link, origin xyz=0.035 0.03 0.02 rpy=0 0 0, axis 1 0 0, mimic joint=small_package_grabber_roller_1_joint multiplier=1 offset=0
- added joint small_package_grabber_roller_3_joint: type continuous, parent small_package_grabber_link, child small_package_grabber_roller_3_link, origin xyz=0.035 -0.02 -0.055 rpy=0 0 0, axis 1 0 0, mimic joint=small_package_grabber_roller_1_joint multiplier=-1 offset=0
- added joint small_package_grabber_roller_4_joint: type continuous, parent small_package_grabber_link, child small_package_grabber_roller_4_link, origin xyz=0.035 -0.03 0.02 rpy=0 0 0, axis 1 0 0, mimic joint=small_package_grabber_roller_1_joint multiplier=-1 offset=0
- added joint small_package_servo_joint: type fixed, parent grr_brain_link, child small_package_sweeper_servo_link, origin xyz=-0.035 0.22 0.025 rpy=0 0 0
- added joint small_package_sweeper_joint: type revolute, parent small_package_sweeper_servo_link, child small_package_sweeper_link, origin xyz=-0.01 0.06 -0.06 rpy=0 0 0, axis 1 0 0, limit lower=-1.57 upper=1.57 effort=100 velocity=0.5
- added joint small_package_sweeper_roller_joint: type continuous, parent small_package_sweeper_link, child small_package_sweeper_roller_link, origin xyz=0 0.05 -0.06 rpy=0 0 0, axis 0 0 1
- joint front_left_mecanum_joint: origin xyz=-0.10075 0.10568 -0.07793 rpy=0 1.5707963267948966 0 -> xyz=-0.10075 0.10568 0 rpy=0 1.5707963267948966 0
- joint front_right_mecanum_joint: origin xyz=0.10075 0.10568 -0.07793 rpy=0 1.5707963267948966 0 -> xyz=0.10075 0.10568 0 rpy=0 1.5707963267948966 0
- joint rear_left_mecanum_joint: origin xyz=-0.10075 -0.10568 -0.07793 rpy=0 -1.5707963267948966 0 -> xyz=-0.10075 -0.10568 0 rpy=0 -1.5707963267948966 0
- joint rear_right_mecanum_joint: origin xyz=0.10075 -0.10568 -0.07793 rpy=0 -1.5707963267948966 0 -> xyz=0.10075 -0.10568 0 rpy=0 -1.5707963267948966 0

File: src/robot_description/urdf/parts/chassis.xacro (robot description, xacro)
@@ -10,5 +10,5 @@
         <origin xyz="0 0 0" rpy="0 0 0"/>
         <geometry>
-          <mesh filename="package://robot_description/meshes/HillCraterDrivebase.stl" scale="0.001 0.001 0.001"/>
+          <mesh filename="package://robot_description/meshes/slim_drivebase.stl" scale="0.001 0.001 0.001"/>
         </geometry>
         <material name="blue"/>

File: src/robot_description/urdf/parts/mecanum_roller.xacro (robot description, xacro)
@@ -28,5 +28,5 @@
         <origin xyz="0 0 0" rpy="0 0 0"/>
         <geometry>
-          <mesh filename="package://robot_description/meshes/rolle2r.stl" scale="0.001 0.001 0.001"/>
+          <mesh filename="package://robot_description/meshes/mechanum_roller.stl" scale="0.001 0.001 0.001"/>
         </geometry>
         <material name="grey"/>
@@ -65,5 +65,5 @@
         <origin xyz="0 0 0" rpy="0 0 0"/>
         <geometry>
-          <mesh filename="package://robot_description/meshes/rolle2r.stl" scale="0.001 0.001 0.001"/>
+          <mesh filename="package://robot_description/meshes/mechanum_roller.stl" scale="0.001 0.001 0.001"/>
         </geometry>
       </collision>

File: src/robot_description/urdf/parts/mecanum_wheel.xacro (robot description, xacro)
@@ -9,5 +9,5 @@
         <origin xyz="0 0 0" rpy="0 0 0"/>
         <geometry>
-          <mesh filename="package://robot_description/meshes/wheel${type}.stl" scale="0.001 0.001 0.001"/>
+          <mesh filename="package://robot_description/meshes/mechanum_wheel_${type}.stl" scale="0.001 0.001 0.001"/>
         </geometry>
         <material name="orange"/>

File: src/robot_description/urdf/robots/examplo.urdf.xacro (robot description, xacro)
@@ -7,4 +7,7 @@
   <xacro:include filename="$(find robot_description)/urdf/parts/mecanum_wheel.xacro"/>
   <xacro:include filename="$(find robot_description)/urdf/parts/mecanum_roller.xacro"/>
+  <xacro:include filename="$(find robot_description)/urdf/parts/small_package_grabber.xacro"/>
+  <xacro:include filename="$(find robot_description)/urdf/parts/small_package_sweeper.xacro"/>
+  <xacro:include filename="$(find robot_description)/urdf/parts/bridge.xacro"/>
   <xacro:include filename="$(find robot_description)/urdf/parts/lidar.xacro"/>
   <xacro:include filename="$(find robot_description)/urdf/parts/zed_cam.xacro"/>
@@ -46,5 +49,5 @@
     pos_x="${wheel_joint_pos_x + wheel_offset}"
     pos_y="${wheel_joint_pos_y}"
-    pos_z="-${wheel_joint_pos_z}"
+    pos_z="-${0}"
     mass="${wheel_weight}"
   />
@@ -57,5 +60,5 @@
     pos_x="-${wheel_joint_pos_x + wheel_offset}"
     pos_y="-${wheel_joint_pos_y}"
-    pos_z="-${wheel_joint_pos_z}"
+    pos_z="-${0}"
     mass="${wheel_weight}"
   />
@@ -68,5 +71,5 @@
     pos_x="-${wheel_joint_pos_x + wheel_offset}"
     pos_y="${wheel_joint_pos_y}"
-    pos_z="-${wheel_joint_pos_z}"
+    pos_z="-${0}"
     mass="${wheel_weight}"
   />
@@ -79,14 +82,26 @@
     pos_x="${wheel_joint_pos_x + wheel_offset}"
     pos_y="-${wheel_joint_pos_y}"
-    pos_z="-${wheel_joint_pos_z}"
+    pos_z="-${0}"
     mass="${wheel_weight}"
   />
-  <xacro:lidar
+  <xacro:small_package_grabber
+    parent="chassis_link"
+    origin="-0.03 0.1 0.03"
+  />
+  <xacro:small_package_sweeper
+    parent="chassis_link"
+    origin="-0.09 -0.14 0.07"
+  />
+  <xacro:bridge
+    parent="chassis_link"
+    origin="0.0 -0.08 0.145"
+  />
+  <!-- <xacro:lidar
     radius="${lidar_radius}"
     length="${lidar_length}"
     pos_y="${lidar_joint_pos_y}"
-  />
-  <xacro:zed_camera parent="chassis_link">
+  /> -->
+  <!-- <xacro:zed_camera parent="chassis_link">
     <origin xyz="0 0.15 0" rpy="0 0 ${pi/2}" />
-  </xacro:zed_camera>
+  </xacro:zed_camera> -->
 </robot>
